Commit message: добавила другие модели роботов

File: urdf/aubo_i10.urdf (robot description, URDF)
Before this commit: robot aubo_i10, 13 links, 12 joints
Links:
- removed link base_gripper
- removed link blue_cube
- removed link finger_left_link
- removed link finger_right_link
- removed link red_cube
- link world: geometry 
Joints:
- removed joint base_gripper_joint
- removed joint cube_joint
- removed joint cube_joint2
- removed joint finger_left_joint
- removed joint finger_right_joint
- joint world_joint: origin xyz=0.0 0.0 0.84 rpy=0.0 0.0 0.0 -> xyz=0.0 0.0 0.0 rpy=0.0 0.0 0.0

File: urdf/xacro/inc/aubo.ros2_control.xacro (robot description, xacro)
@@ -1,8 +1,5 @@
 <?xml version="1.0"?>
 <robot xmlns:xacro="http://www.ros.org/wiki/xacro">
-  <xacro:macro name="aubo_ros2_control" params="name prefix use_fake_hardware:=false robot_ip config">
- <xacro:property name="initial_positions" value="${xacro.load_yaml(config)['initial_positions']}"/>
- <xacro:property name="upper_limits" value="${xacro.load_yaml(config)['upper_limits']}"/>
- <xacro:property name="lower_limits" value="${xacro.load_yaml(config)['lower_limits']}"/>
+  <xacro:macro name="aubo_ros2_control" params="name prefix use_fake_hardware:=false robot_ip">
     <ros2_control name="${name}" type="system">
       <hardware>
@@ -90,25 +87,4 @@
       </joint>
     </ros2_control>
-     <ros2_control name="gripper_ros2_control" type="system">
-            <hardware>
-                 <plugin>gripper_driver/GripperHardwareInterface</plugin>
-            </hardware>
-            <joint name="finger_left_joint">
-                <command_interface name="position"/>
-                <state_interface name="position">
-                  <param name="initial_value">${initial_positions['finger_left_link']}</param>
-                  <param name="upper_limits">${upper_limits['finger_left_link']}</param>
-                  <param name="lower_limits">${lower_limits['finger_left_link']}</param>
-                </state_interface>
-            </joint>
-            <joint name="finger_right_joint">
-                <command_interface name="position"/>
-                <state_interface name="position">
-                  <param name="initial_value">${initial_positions['finger_right_link']}</param>
-                  <param name="upper_limits">${upper_limits['finger_right_link']}</param>
-                  <param name="lower_limits">${lower_limits['finger_right_link']}</param>
-                </state_interface>
-            </joint>
-     </ros2_control>
   </xacro:macro>
 </robot>

File: urdf/xacro/inc/aubo_ros2.xacro (robot description, xacro)
@@ -4,5 +4,5 @@
   <xacro:arg name="robot_ip" default="None"/>
     <xacro:property name="robot_ip" value="$(arg robot_ip)"/>
-  <xacro:arg name="aubo_type" default="aubo_i10"/>
+  <xacro:arg name="aubo_type" default="None"/>
     <xacro:property name="aubo_type" value="$(arg aubo_type)"/>
   <xacro:arg name="use_fake_hardware" default="true"/>
@@ -13,5 +13,4 @@
     aubo_type="${aubo_type}"/>
   <!-- ros2_control -->
-   <xacro:arg name="config_file" default="config_file.yaml" />
   <xacro:include filename="$(find aubo_description)/urdf/xacro/inc/aubo.ros2_control.xacro" />
   <xacro:aubo_ros2_control
@@ -19,6 +18,4 @@
     prefix=""
     use_fake_hardware="${use_fake_hardware}"
-    robot_ip="${robot_ip}"
-    config = "$(arg config_file)"
-    />
+    robot_ip="${robot_ip}"/>
 </robot>

File: urdf/xacro/inc/aubo_ros2_macro.xacro (robot description, xacro)
@@ -3,5 +3,4 @@
   <xacro:macro name="aubo_robot" params="aubo_type transmission_hw_interface">
     <xacro:include filename="$(find aubo_description)/urdf/${aubo_type}.urdf.xacro" />
-    <!-- <xacro:include filename="$(find environment_description)/urdf/crane_motor/table_macro.xacro" />  -->
     <joint name="ee_fixed_joint" type="fixed">
       <parent link="wrist3_Link" />
